File: PWMGenerator_bpham5/_autosave-PWMGenerator_bpham5.kicad_sch (KiCad schematic)
At the start: 29 parts, among them J1 Conn_01x03, Q1 2N3904, Q2 2N3904, Q3 2N3906, Q4 2N3906, SW1 SW_SPST, U1 LM7805_TO220, U2 LM339

Commit message: partbcompleted
Parts:
- added R11: NANOSMDC016F-2, NANOSMDC016F-2:RESC3115X65N, symbol NANOSMDC016F-2:NANOSMDC016F-2
- C1: value C_US -> 220uF; footprint (none) -> Capacitor_THT:CP_Radial_D4.0mm_P2.00mm
- C2: value C_US -> 10uF; footprint (none) -> Capacitor_THT:CP_Radial_D4.0mm_P2.00mm
- C3: value C -> 0.1uF
- SW1: footprint (none) -> Button_Switch_SMD:SW_DIP_SPSTx01_Slide_6.7x4.1mm_W6.73mm_P2.54mm_LowProfile_JPin
Changed lines of the file:
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@@
 			)
 		)
-		(property "Footprint" ""
+		(property "Footprint" "Button_Switch_SMD:SW_DIP_SPSTx01_Slide_6.7x4.1mm_W6.73mm_P2.54mm_LowProfile_JPin"
 			(at 26.67 100.33 0)
 			(effects
@@
 			)
 		)
-		(property "Value" "C_US"
+		(property "Value" "10uF"
 			(at 144.78 109.4739 0)
 			(effects
@@
 			)
 		)
-		(property "Footprint" ""
+		(property "Footprint" "Capacitor_THT:CP_Radial_D4.0mm_P2.00mm"
 			(at 140.97 107.95 0)
 			(effects
@@
 			)
 		)
-		(property "Datasheet" ""
+		(property "Datasheet" "https://www.cde.com/resources/catalogs/SVF.pdf"
 			(at 140.97 107.95 0)
 			(effects
@@
 			)
 		)
-		(property "Value" "C"
+		(property "Value" "0.1uF"
 			(at 193.04 130.8099 0)
 			(effects
@@
 	)
 	(symbol
+		(lib_id "NANOSMDC016F-2:NANOSMDC016F-2")
+		(at 82.55 55.88 0)
+		(unit 1)
+		(exclude_from_sim no)
+		(in_bom yes)
+		(on_board yes)
+		(dnp no)
+		(fields_autoplaced yes)
+		(property "Reference" "R11"
+			(at 82.55 49.53 0)
+			(effects
+				(font
+					(size 1.27 1.27)
+				)
+			)
+		)
+		(property "Value" "NANOSMDC016F-2"
+			(at 82.55 52.07 0)
+			(effects
+				(font
+					(size 1.27 1.27)
+				)
+			)
+		)
+		(property "Footprint" "NANOSMDC016F-2:RESC3115X65N"
+			(at 82.55 55.88 0)
+			(effects
+				(font
+					(size 1.27 1.27)
+				)
+				(justify bottom)
+				(hide yes)
+			)
+		)
+		(property "Datasheet" ""
+			(at 82.55 55.88 0)
+			(effects
+				(font
+					(size 1.27 1.27)
+				)
+				(hide yes)
+			)
+		)
+		(property "Description" ""
+			(at 82.55 55.88 0)
+			(effects
+				(font
+					(size 1.27 1.27)
+				)
+				(hide yes)
+			)
+		)
+		(pin "1"
+		)
+		(pin "2"
+		)
+		(instances
+			(project ""
+				(path "/0859a153-53e5-453d-9797-4636ab796f1d"
+					(reference "R11")
+					(unit 1)
+				)
+			)
+		)
+	)
+	(symbol
 		(lib_id "Device:R_US")
 		(at 158.75 101.6 0)
@@
 			)
 		)
-		(property "Value" "C_US"
+		(property "Value" "220uF"
 			(at 102.87 110.7439 0)
 			(effects
@@
 			)
 		)
-		(property "Footprint" ""
+		(property "Footprint" "Capacitor_THT:CP_Radial_D4.0mm_P2.00mm"
 			(at 99.06 109.22 0)
 			(effects
@@
 			)
 		)
-		(property "Datasheet" ""
+		(property "Datasheet" "https://www.vishay.com/docs/28321/136rvi.pdf"
 			(at 99.06 109.22 0)
 			(effects
