File: PWMGenerator_bpham5/PWMGenerator_bpham5.kicad_sch (KiCad schematic)
At the start: 0 parts

Commit message: PCB PART A
Parts:
- added C1, C2: C_US, symbol Device:C_US
- added C3: C, symbol Device:C
- added D1, D2, D3, D4, D6: 1N4005, Diode_THT:D_DO-41_SOD81_P10.16mm_Horizontal, symbol Diode:1N4005
- added D5: SFH4550, LED_THT:LED_D5.0mm_IRGrey, symbol LED:SFH4550
- added J1: Conn_01x03, symbol Connector_Generic:Conn_01x03
- added Q1, Q2: 2N3904, Package_TO_SOT_THT:TO-92_Inline, symbol Transistor_BJT:2N3904
- added Q3, Q4: 2N3906, Package_TO_SOT_THT:TO-92_Inline, symbol Transistor_BJT:2N3906
- added R1, R10, R2, R3, R4, R5, R6, R7, R8, R9: R_US, symbol Device:R_US
- added RV1: R_Potentiometer_US, symbol Device:R_Potentiometer_US
- added SW1: SW_SPST, symbol Switch:SW_SPST
- added U1: LM7805_TO220, Package_TO_SOT_THT:TO-220-3_Vertical, symbol Regulator_Linear:LM7805_TO220
- added U2: LM339, symbol Comparator:LM339
- added V1: VSIN, symbol Simulation_SPICE:VSIN
Connections:
- new net: Q1.2 (B), R1.2
- new net: Q1.3 (C), Q2.2 (B), R4.2
- new net: D1.1 (K), D2.1 (K), D6.2 (A), R1.1, R2.1
- new net: C2.1, J1.1 (Pin_1), Q4.1 (E), R3.1, R4.1, R5.1, R6.1, R7.1, U1.3 (VO)
- new net: Q4.2 (B), R9.2
- new net: J1.2 (Pin_2), Q4.3 (C), R10.2
- new net: R7.2, RV1.3, U2.5 (+)
- new net: C1.1, D6.1 (K), U1.1 (VI)
- new net: R9.1, U2.2
- new net: SW1.1 (A), V1.1
- new net: D2.2 (A), D3.1 (K), SW1.2 (B)
- new net: C3.1, Q2.3 (C), Q3.3 (C), U2.4 (-)
- new net: D1.2 (A), D4.1 (K), V1.2
- new net: Q3.1 (E), R6.2
- new net: D5.2 (A), R3.2
- new net: Q3.2 (B), R5.2, R8.1
- new net GND: C1.2, C2.2, C3.2, D3.2 (A), D4.2 (A), D5.1 (K), J1.3 (Pin_3), Q1.1 (E), Q2.1 (E), R10.1, R2.2, R8.2, RV1.1, RV1.2, U1.2 (GND)
Other:
- company: (none) -> NAIT CNT
- title: (none) -> CMPE2150 PWM Generator - bpham5

Commit message: part b completed
Parts:
- C1: value C_US -> 220uF; footprint (none) -> Capacitor_THT:CP_Radial_D4.0mm_P2.00mm
- C2: value C_US -> 10uF; footprint (none) -> Capacitor_THT:CP_Radial_D4.0mm_P2.00mm
- C3: value C -> 0.1uF; footprint (none) -> Capacitor_SMD:C_0805_2012Metric
- D1, D2, D3, D4, D6: footprint Diode_THT:D_DO-41_SOD81_P10.16mm_Horizontal -> Diode_SMD:D_0805_2012Metric
- D5: footprint LED_THT:LED_D5.0mm_IRGrey -> LED_THT:LED_D5.0mm_GREEN
- J1: footprint (none) -> Connector_PinHeader_2.54mm:PinHeader_1x03_P2.54mm_Vertical
- Q1, Q2, Q3, Q4: footprint Package_TO_SOT_THT:TO-92_Inline -> Package_TO_SOT_SMD:SOT-23
- R1, R7: value R_US -> 2.2k; footprint (none) -> Resistor_SMD:R_0805_2012Metric
- R10: value R_US -> 180; footprint (none) -> Resistor_SMD:R_0805_2012Metric
- R2: value R_US -> 1M; footprint (none) -> Resistor_SMD:R_0805_2012Metric
- R3: value R_US -> 330; footprint (none) -> Resistor_SMD:R_0805_2012Metric
- R4: value R_US -> 10k; footprint (none) -> Resistor_SMD:R_0805_2012Metric
- R5: value R_US -> 220k; footprint (none) -> Resistor_SMD:R_0805_2012Metric
- R6: value R_US -> 22k; footprint (none) -> Resistor_SMD:R_0805_2012Metric
- R8: value R_US -> 390k; footprint (none) -> Resistor_SMD:R_0805_2012Metric
- R9: value R_US -> 8.2k; footprint (none) -> Resistor_SMD:R_0805_2012Metric
- RV1: footprint (none) -> Potentiometer_THT:Potentiometer_ACP_CA9-V10_Vertical_Hole
- SW1: footprint (none) -> Button_Switch_SMD:SW_DIP_SPSTx01_Slide_6.7x4.1mm_W6.73mm_P2.54mm_LowProfile_JPin
- U1: footprint Package_TO_SOT_THT:TO-220-3_Vertical -> Package_TO_SOT_THT:TO-220-3_Horizontal_TabDown
- U2: footprint (none) -> Package_SO:SOIC-14_3.9x8.7mm_P1.27mm
- V1: footprint (none) -> Connector_BarrelJack:BarrelJack_CUI_PJ-063AH_Horizontal; symbol Simulation_SPICE:VSIN -> Connector:Barrel_Jack
Connections:
- net GND: now also R1.1, V1.2; no longer R2.2
- net at Q1.2 (B): now also R2.2; no longer R1.2
- net at D1.1 (K), D2.1 (K), D6.2 (A)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: now also R1.2; no longer R1.1
- net at SW1.1 (A), V1.1: now also D1.2 (A), D4.1 (K)
Other:
- moved on the sheet: R1, R2

Commit message: part b fixed
Parts:
- removed V1: VSIN, Connector_BarrelJack:BarrelJack_CUI_PJ-063AH_Horizontal, symbol Connector:Barrel_Jack
- added J2: Barrel_Jack, Connector_BarrelJack:BarrelJack_CUI_PJ-063AH_Horizontal, symbol Connector:Barrel_Jack
- added R11: NANOSMDC016F-2, NANOSMDC016F-2:RESC3115X65N, symbol NANOSMDC016F-2:NANOSMDC016F-2
Connections:
- net at D1.2 (A), D4.1 (K): now also J2.2; no longer SW1.1 (A)
- net at D2.2 (A), D3.1 (K): now also R11.2; no longer SW1.2 (B)
- new net: J2.1, SW1.1 (A)
- new net: R11.1, SW1.2 (B)
