File: PWMGenerator_bpham5/PWMGenerator_bpham5.kicad_pcb (KiCad board)
At the start: 2 copper layers, 30 parts, among them J1 Conn_01x03, J2 Barrel_Jack, Q1 2N3904, Q2 2N3904, Q3 2N3906, Q4 2N3906, SW1 SW_SPST, U1 LM7805_TO220, U2 LM339

Commit message: PCB IN PROGRESS
Parts:
- U1: moved to B.Cu
- moved D5 141.9 mm to (49.7, 30.9)
- moved R11 108.8 mm to (54.0, 39.9)
- moved J2 107.8 mm to (54.0, 69.4)
- moved SW1 102.4 mm to (54.0, 50.9), turned to 90 degrees
- moved D6 84.9 mm to (100.6, 39.5)
- moved D2 81.2 mm to (71.1, 97.5)
- moved D1 78.2 mm to (76.0, 77.5), turned to 180 degrees
- moved C1 74.1 mm to (118.0, 41.0)
- moved D4 66.9 mm to (89.6, 80.5)
- moved C2 65.3 mm to (142.0, 40.0)
- moved R8 64.2 mm to (112.9, 100.5), turned to 180 degrees
- moved R7 64.0 mm to (112.1, 93.5), turned to 180 degrees
- moved R6 63.4 mm to (112.1, 87.5), turned to 180 degrees
- moved D3 62.8 mm to (89.6, 97.0)
- moved R1 61.0 mm to (112.9, 56.0), turned to 180 degrees
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Other:
- board outline added: 148 x 82.5 mm

Commit message: PCB ALMOST COMPLETED
Parts:
- moved R9 23.1 mm to (145.4, 97.0)
- moved R10 22.3 mm to (159.5, 85.5)
- moved J2 12.8 mm to (63.5, 77.9)
- moved Q2 12.8 mm to (130.9, 84.6)
- moved C1 12.8 mm to (127.5, 49.5)
- moved C2 12.8 mm to (151.5, 48.5)
- moved D6 12.8 mm to (110.1, 48.0)
- moved J1 12.8 mm to (182.5, 69.9)
- moved RV1 12.8 mm to (177.0, 48.0)
- moved U1 12.8 mm to (143.5, 55.7)
- moved D5 12.8 mm to (59.2, 39.4)
- moved C3 12.8 mm to (141.0, 75.5)
- moved D1 12.8 mm to (85.5, 86.0)
- moved D2 12.8 mm to (80.6, 106.0)
- moved D3 12.8 mm to (99.1, 105.5)
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Routing:
- net Net-(J1-Pin_1): track 0.00 -> 62.5 mm
- net Net-(U2A-+): track 0.00 -> 35.6 mm
- net Net-(J1-Pin_2): track 0.00 -> 33.8 mm
- net Net-(Q2-C): track 0.00 -> 26.3 mm
- net Net-(Q4-B): track 0.00 -> 23.2 mm
- net Net-(R9-Pad1): track 0.00 -> 12.3 mm
- net GND: track 0.00 -> 0.70 mm, vias 0 -> 6
- added copper zone on B.Cu, net GND
- added copper zone on F.Cu, net VCC
Other:
- board outline removed
