File: PWMGenerator_bpham5 - Copy/PWMGenerator_bpham5.kicad_sch (KiCad schematic)
At the start: 30 parts, among them J1 Conn_01x03, J2 Barrel_Jack, Q1 2N3904, Q2 2N3904, Q3 2N3906, Q4 2N3906, SW1 SW_SPST, U1 LM7805_TO220, U2 LM339

Commit message: PROJECT C STARTED
Parts:
- D5: footprint LED_THT:LED_D5.0mm_IRGrey -> LED_THT:LED_D5.0mm_GREEN
- R11: footprint NANOSMDC016F_2:RESC3115X65N -> NANOSMDC016F-2:RESC3115X65N
Changed lines of the file:
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@@
 			)
 		)
-		(property "Footprint" "LED_THT:LED_D5.0mm_IRGrey"
+		(property "Footprint" "LED_THT:LED_D5.0mm_GREEN"
 			(at 154.305 113.03 0)
 			(effects
@@
 			)
 		)
-		(property "Footprint" "NANOSMDC016F_2:RESC3115X65N"
+		(property "Footprint" "NANOSMDC016F-2:RESC3115X65N"
 			(at 45.72 82.55 0)
 			(effects
